File: OpenCAPI_PCIe_x4_Host_and_Endpoint.kicad_pcb (KiCad board)
At the start: 4 copper layers, 65.9 x 40.5 mm, 35 parts, among them J1 OpenCAPI_AAC_Host, J2 Conn_01x06, J3 Bus_PCI_Express_x4, J4 Bus_PCI_Express_x4, J7 CLK_P, J8 CLK_N, U1 SY75572L, U2 DSC1124B

Commit message: First Revision Complete
Parts:
- removed R7: DNP, Resistor_SMD:R_0603_1608Metric_Pad0.98x0.95mm_HandSolder
- added TP4: 3V3, TestPoint:TestPoint_THTPad_D1.0mm_Drill0.5mm, F.Cu at (60.0, 79.5)
- added TP5: 3V3, TestPoint:TestPoint_THTPad_D1.0mm_Drill0.5mm, F.Cu at (97.6, 76.5)
- added TP6: nPERST, TestPoint:TestPoint_THTPad_D1.0mm_Drill0.5mm, F.Cu at (107.8, 76.5)
- added TP7: nPERST, TestPoint:TestPoint_THTPad_D1.0mm_Drill0.5mm, F.Cu at (64.5, 78.2)
- moved J2 6.54 mm to (109.0, 79.0)
- moved L2 3.27 mm to (63.5, 52.1)
- moved TP2 1.51 mm to (69.8, 78.5)
- moved L1 0.60 mm to (72.1, 61.0)
- moved TP1 0.50 mm to (52.5, 79.8)
- moved R2 0.40 mm to (73.5, 61.0)
- moved R1 0.28 mm to (71.2, 71.4)
- moved JP1 0.25 mm to (67.8, 55.2)
Connections:
- J1 pad A21: nPERST -> nPERST_JMP
- J2 pad 1: GND -> nPERST_JMP
- J2 pad 3: SCL -> SDA
- J2 pad 4: SDA -> GND
- J2 pad 5: nPERST -> SCL
- J3 pad B31: Net-(J3-~{PRSNT1}) -> Net-(J3-~{PRSNT2}-PadB31)
- TP3 pad 1: Net-(J3-~{PRSNT1}) -> Net-(J3-~{PRSNT2}-PadB31)
Routing:
- net GND: track 357.9 -> 1255.6 mm, vias 89 -> 193
- net nTRST: track 0.00 -> 42.7 mm
- net +3.3VA: track 0.00 -> 42.2 mm
- net nWAKE: track 0.00 -> 42.2 mm
- net nPERST_JMP: track 0.00 -> 35.6 mm, vias 0 -> 2
- net +12V: track 147.6 -> 112.4 mm
- net SCL: track 0.00 -> 34.0 mm, vias 0 -> 2
- net SDA: track 0.00 -> 32.7 mm, vias 0 -> 2
- net Rx1_N: track 43.9 -> 73.0 mm
- net Rx1_P: track 44.1 -> 72.6 mm
- net PRE_DETECT: track 0.00 -> 25.3 mm, vias 0 -> 3
- net Rx0_N: track 49.2 -> 73.1 mm
- net Tx6_N: track 32.6 -> 55.8 mm
- net Tx6_P: track 33.4 -> 56.5 mm
- net +3.3V: track 117.5 -> 94.6 mm, vias 2 -> 4
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- added copper zone on B.Cu, net GND
- added copper zone on F.Cu, net GND
- added copper zone on In1.Cu, net GND
- added copper zone on In2.Cu, net GND
Other:
- board size 65.9 x 40.5 mm -> 59.7 x 40.5 mm
- board text added: "1"
- board text added: "4"
- board text added: "OpenCAPI to PCIe x4 Host and Endpoint"
- board text removed: "OpenCAPI-Compatible SlimSAS 8x Breakout"
