File: OpenCAPI_PCIe_x4_Host_and_Endpoint.kicad_sch (KiCad schematic)
At the start: 35 parts, among them J1 OpenCAPI_AAC_Host, J2 Conn_01x06, J3 Bus_PCI_Express_x4, J4 Bus_PCI_Express_x4, J7 CLK_P, J8 CLK_N, U1 SY75572L, U2 DSC1124B

Commit message: First Revision Complete
Parts:
- removed R7: DNP, Resistor_SMD:R_0603_1608Metric_Pad0.98x0.95mm_HandSolder, symbol Device:R_Small_US
- added TP4, TP5: 3V3, TestPoint:TestPoint_THTPad_D1.0mm_Drill0.5mm, symbol Connector:TestPoint
- added TP6, TP7: nPERST, TestPoint:TestPoint_THTPad_D1.0mm_Drill0.5mm, symbol Connector:TestPoint
Connections:
- net +3.3V: now also TP4.1, TP5.1
- net GND: now also J2.4 (Pin_4); no longer J2.1 (Pin_1)
- net SCL: now also J2.5 (Pin_5); no longer J2.3 (Pin_3)
- net SDA: now also J2.3 (Pin_3); no longer J2.4 (Pin_4)
- net nPERST: now also TP7.1; no longer J1.A21 (INT_RST), J2.5 (Pin_5)
- net at J3.A1 (~{PRSNT1}), TP1.1: no longer J3.B31 (~{PRSNT2}), TP3.1
- new net: J3.B31 (~{PRSNT2}), TP3.1
- new net nPERST_JMP: J1.A21 (INT_RST), J2.1 (Pin_1), TP6.1
Other:
- note added: "Clock Source Selection and Distribution"
- note added: "Same pinout order as a TC74A0-3.3VAT Temperature Sensor"
- note added: "Use a Wire Jumper to Connect"
- note added: "Wire Jumpers"
- note removed: "Clock Source Select and Distribution"
- moved on the sheet: J2
